File: nabijecka.brd (EAGLE design)
At the start: 93 x 75 mm, 69 parts, among them T1 BD244C, T2 BD244C, T3 BC556, T4 BC556, T5 BD244C, T6 BC556, U1 TINY45-20-DIP, X1 04-JST-B4B-XH-A

Commit message: Add schema in PDF. Rename files.
Parts:
- C10: value (none) -> 100n
Changed lines of the file:
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@@
 <element name="R7" library="resistor" package="R1206" value="47K" x="26.9494" y="3.1242" rot="MR0"/>
 <element name="R8" library="resistor" package="R1206" value="10K" x="22.9362" y="4.5212" rot="MR90"/>
-<element name="C10" library="resistor" package="C1206" value="" x="16.3322" y="4.572" rot="MR90"/>
+<element name="C10" library="resistor" package="C1206" value="100n" x="16.3322" y="4.572" rot="MR90"/>
 <element name="T1" library="transistor" package="TO220" value="BD244C" x="35.3556" y="52.8538"/>
 <element name="D3" library="diode" package="SOD80C" value="1N4148" x="29.1592" y="45.339" rot="MR90"/>
